File: pwr-v1/pwr-v1.kicad_pcb (KiCad board)
At the start: 2 copper layers, 310 x 50 mm, 86 parts, among them SW101 SW_SPST, U101 TYPE-C-31-M-12, U102 SK-3296S-01-L1, U103 CH224K, U104 AMS1117-5.0, U105 LM2595S-12, U106 LM2595S-12

Commit message: Fix bad edgecuts
Other:
- outline, holes or cut-outs redrawn
Changed lines of the file:
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@@
     (pad "2" smd rect (at 4.95 0 90) (size 2.9 5.4) (layers "F.Cu" "F.Paste" "F.Mask")
       (net 3 "+12V") (pintype "passive"))
-    (model "${KICAD6_3DMODEL_DIR}/Inductor_SMD.3dshapes/L_12x12mm_H6mm.wrl"
+    (model "/Users/gazda/Documents/Mnau-Labs/KiCad Libraries/PWR1LCSC1/footprint/packages3d/IND-SMD_L12.3-W12.3_SMDRI127.wrl"
       (offset (xyz 0 0 0))
       (scale (xyz 1 1 1))
@@
       (net 24 "Net-(R102-Pad1)") (pinfunction "3") (pintype "unspecified"))
     (model "/Users/gazda/Documents/Mnau-Labs/KiCad Libraries/PWR1LCSC1/footprint/packages3d/SW-SMD_3P-P1.50_L2.7-W6.6.wrl"
-      (offset (xyz 0 0 0))
+      (offset (xyz 0 -0.25 0))
       (scale (xyz 1 1 1))
       (rotate (xyz 0 0 -180))
@@
     (pad "B12" smd rect locked (at -3.051054 -3.7841 270) (size 0.3 1.3) (layers "F.Cu" "F.Paste" "F.Mask")
       (net 4 "GND") (pinfunction "GND") (pintype "unspecified"))
-    (model "/Users/gazda/Documents/Mnau-Labs/KiCad Libraries/PWR1LCSC1/footprint/packages3d/USB-C_SMD-TYPE-C-31-M-12.wrl"
-      (offset (xyz 0 0 0))
-      (scale (xyz 1 1 1))
-      (rotate (xyz 0 0 -180))
+    (model "/Users/gazda/Documents/Mnau-Labs/KiCad Libraries/PWR1LCSC1/footprint/packages3d/HRO_TYPE-C-31-M-12.step"
+      (offset (xyz -4.5 -3.75 0))
+      (scale (xyz 1 1 1))
+      (rotate (xyz 0 0 0))
     )
   )
@@
     (pad "2" smd rect (at 4.95 0) (size 2.9 5.4) (layers "F.Cu" "F.Paste" "F.Mask")
       (net 4 "GND") (pintype "passive"))
-    (model "${KICAD6_3DMODEL_DIR}/Inductor_SMD.3dshapes/L_12x12mm_h8mm.wrl.html"
+    (model "/Users/gazda/Documents/Mnau-Labs/KiCad Libraries/PWR1LCSC1/footprint/packages3d/IND-SMD_L12.3-W12.3_SMDRI127.wrl"
       (offset (xyz 0 0 0))
       (scale (xyz 1 1 1))
@@
   (gr_line (start 39.6 73.2) (end 304.4 73.2) (layer "F.SilkS") (width 2))
   (gr_arc (start 305 39.25) (mid 308.535534 40.714466) (end 310 44.25) (layer "Edge.Cuts") (width 0.15))
-  (gr_line (start 0 39.27) (end 305 39.25) (layer "Edge.Cuts") (width 0.15))
+  (gr_line (start 0 39.25) (end 305 39.25) (layer "Edge.Cuts") (width 0.15))
   (gr_arc (start 310 84.25) (mid 308.535534 87.785534) (end 305 89.25) (layer "Edge.Cuts") (width 0.15))
-  (gr_line (start 305 89.25) (end 0 89.175) (layer "Edge.Cuts") (width 0.15))
+  (gr_line (start 305 89.25) (end 0 89.25) (layer "Edge.Cuts") (width 0.15))
   (gr_line (start 310 44.25) (end 310 84.25) (layer "Edge.Cuts") (width 0.15))
-  (gr_line (start 0 39.27) (end 0 89.175) (layer "Edge.Cuts") (width 0.2))
+  (gr_line (start 0 39.25) (end 0 89.25) (layer "Edge.Cuts") (width 0.2))
   (gr_rect (start 0 0) (end 326 128.5) (layer "User.1") (width 0.15) (fill none))
   (gr_rect (start 326 0) (end 327.6 128.5) (layer "User.3") (width 0.15) (fill solid))
